File: pcb/gpib_adapter.sch (KiCad schematic (older format))
At the start: 27 parts, among them IC1 ATMEGA16U4, P1 ISP, P2 USB, P3 GPIO, P4 UART, P5 GPIB, P6 PWR_JMP, U1 SN75160, U2 SN75161

Commit message: change processor
Parts:
- removed C1: 100n, symbol C
- removed IC1: ATMEGA16U4, TQFP44, symbol ATMEGA16U4
- removed L1: Ferrite, symbol INDUCTOR
- removed R4: 2.2k, symbol R
- added D? (x3): PWR, symbol LED-RESCUE-gpib_adapter
- added R? (x3): R, symbol R-RESCUE-gpib_adapter
- added U?: FT230XQ, QFN-16, symbol FT230XQ
- added U?: AT90CAN128-A, TQFP64, symbol AT90CAN128-A
- C2, C3, C4, C5, C6, C7, C8: symbol C -> C-RESCUE-gpib_adapter
- D1: symbol LED -> LED-RESCUE-gpib_adapter
- R1, R2, R3, R5, R6, R7: symbol R -> R-RESCUE-gpib_adapter
Connections:
- net labels added: GPIO0, GPIO6, GPIO7
- wire segments 142 -> 171
Other:
- moved on the sheet: C2, C4, C7, C8, P1, P2, P3, P5, R2, R3, R5, R6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

Commit message: adding some code
Parts:
- removed D1: PWR, symbol LED-RESCUE-gpib_adapter
- removed D2: LED_X2, symbol LED_X2
- removed P1: ISP, symbol CONN_3X2
- removed P4: UART, symbol CONN_4
- removed P6: PWR_JMP, symbol CONN_4
- added C1: 22µ, Capacitors_SMD:c_elec_5x5.3, symbol C-RESCUE-gpib_adapter
- added CON1: AVR-ISP-6, w_pin_strip:pin_socket_3x2, symbol AVR-ISP-6
- added J1: HEADER_2, w_pin_strip:pin_socket_2, symbol HEADER_2
- added R10, R11, R12, R13, R14, R15, R16, R17, R18, R19, R20, R24, R25, R4, R8, R9: R, Resistors_SMD:R_0805, symbol R-RESCUE-gpib_adapter
- C2, C3, C5, C6, C7, C8: footprint (none) -> Capacitors_SMD:C_0805
- C4: footprint (none) -> Capacitors_SMD:C_1206
- D1, D2, D3: renamed from D?; footprint (none) -> Capacitors_SMD:C_0805
- P2: footprint (none) -> w_conn_pc:conn_usb_B
- P3: footprint (none) -> w_pin_strip:pin_socket_3x2
- P5: footprint (none) -> w_pin_strip:pin_socket_12x2
- R1: value 2.2k -> R; footprint (none) -> Resistors_SMD:R_0805
- R2, R3, R5, R7: footprint (none) -> Resistors_SMD:R_0805
- R21, R22, R23: renamed from R?; footprint (none) -> Resistors_SMD:R_0805
- R6: footprint (none) -> Resistors_SMD:R_2010
- U1, U2: footprint (none) -> Housings_SOIC:SOIC-20_7.5x12.8mm_Pitch1.27mm
- U3: renamed from U?; footprint QFN-16 -> Housings_DFN_QFN:QFN-16-1EP_4x4mm_Pitch0.65mm
- U4: renamed from U?; footprint TQFP64 -> Housings_QFP:LQFP-64_14x14mm_Pitch0.8mm
Connections:
- net labels added: MISO, MOSI, PE, RESET, SCK
- net labels removed: GPIO0, GPIO6, GPIO7, Res, VCC, VDD
- wire segments 171 -> 215
- no-connect marks 0 -> 14
Other:
- moved on the sheet: C2, C3, C4, C5, C6, C7, C8, D1, D2, D3, P2, P3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

Commit message: changing project structure
Connections:
- wire segments 215 -> 213
- no-connect marks 14 -> 16
Changed lines of the file:
@@
 Text Label 10200 6900 0    60   ~ 0
 DC
-Text Label 9400 4625 0    60   ~ 0
-MISO
 Text Label 9400 4725 0    60   ~ 0
 GPIO2
@@
 	9675 4725 9775 4625
 Entry Wire Line
-	9675 4625 9775 4525
-Entry Wire Line
-	9675 4525 9775 4425
-Entry Wire Line
 	9675 4425 9775 4325
 Entry Wire Line
@@
 	1    0    0    -1
 $EndComp
-Text Label 9400 4525 0    60   ~ 0
-MOSI
 Text Label 9400 4425 0    60   ~ 0
 SCK
@@
 Wire Wire Line
 	9375 4425 9675 4425
-Wire Wire Line
-	9375 4525 9675 4525
-Wire Wire Line
-	9375 4625 9675 4625
 Wire Wire Line
 	9375 4725 9675 4725
@@
 Text Label 9375 8200 0    60   ~ 0
 RESET
+Text Label 6400 6225 0    60   ~ 0
+MISO
+Text Label 6400 6125 0    60   ~ 0
+MOSI
+NoConn ~ 9375 4525
+NoConn ~ 9375 4625
 $EndSCHEMATC

Commit message: fix hardware issues
Connections:
- wire segments 213 -> 219
Changed lines of the file:
@@
 L GND-RESCUE-gpib_adapter #PWR02
 U 1 1 4FFC9BA8
-P 13550 4900
-F 0 "#PWR02" H 13550 4900 30  0001 C CNN
-F 1 "GND" H 13550 4830 30  0001 C CNN
-F 2 "" H 13550 4900 60  0001 C CNN
-F 3 "" H 13550 4900 60  0001 C CNN
-	1    13550 4900
-	1    0    0    -1
-$EndComp
+P 14500 4900
+F 0 "#PWR02" H 14500 4900 30  0001 C CNN
+F 1 "GND" H 14500 4830 30  0001 C CNN
+F 2 "" H 14500 4900 60  0001 C CNN
+F 3 "" H 14500 4900 60  0001 C CNN
+	1    14500 4900
+	1    0    0    -1
+$EndComp
+Text Label 9400 6325 0    60   ~ 0
+RXD
 Text Label 9400 6425 0    60   ~ 0
-RXD
-Text Label 9400 6325 0    60   ~ 0
 TXD
 Entry Wire Line
@@
 Entry Wire Line
 	14750 3750 14850 3650
-Entry Wire Line
-	14750 4250 14850 4150
-Entry Wire Line
-	14750 4350 14850 4250
 $Comp
 L CONN_5 P2
@@
 Entry Wire Line
 	11950 4250 12050 4150
-Text Label 13200 3650 0    60   ~ 0
+Text Label 13250 3650 0    60   ~ 0
 DIO1 B
-Text Label 14400 3650 0    60   ~ 0
+Text Label 13250 3750 0    60   ~ 0
 DIO2 B
-Text Label 13200 3750 0    60   ~ 0
+Text Label 13250 3850 0    60   ~ 0
 DIO3 B
-Text Label 14400 3750 0    60   ~ 0
+Text Label 13250 3950 0    60   ~ 0
 DIO4 B
-Text Label 13200 4250 0    60   ~ 0
+Text Label 14425 3650 0    60   ~ 0
 DIO5 B
-Text Label 14400 4250 0    60   ~ 0
+Text Label 14425 3750 0    60   ~ 0
 DIO6 B
-Text Label 13200 4350 0    60   ~ 0
+Text Label 14425 3850 0    60   ~ 0
 DIO7 B
-Text Label 14400 4350 0    60   ~ 0
+Text Label 14425 3950 0    60   ~ 0
 DIO8 B
 Entry Wire Line
@@
 Text Label 11600 6550 0    60   ~ 0
 SRQ B
-Text Label 13200 3850 0    60   ~ 0
+Text Label 13250 4050 0    60   ~ 0
 EOI B
-Text Label 13200 3950 0    60   ~ 0
+Text Label 13250 4250 0    60   ~ 0
 NRFD B
-Text Label 14400 3850 0    60   ~ 0
+Text Label 13250 4150 0    60   ~ 0
 DAV B
-Text Label 13200 4050 0    60   ~ 0
+Text Label 13250 4450 0    60   ~ 0
 IFC B
-Text Label 14400 4050 0    60   ~ 0
+Text Label 13250 4550 0    60   ~ 0
 SRQ B
-Text Label 13200 4150 0    60   ~ 0
+Text Label 13250 4650 0    60   ~ 0
 ATN B
-Text Label 14400 3950 0    60   ~ 0
+Text Label 13250 4350 0    60   ~ 0
 NDAC B
 Entry Wire Line
@@
 	0    -1   -1   0
 $EndComp
-Text Label 13200 4450 0    60   ~ 0
+Text Label 14450 4050 0    60   ~ 0
 REN B
 Entry Wire Line
@@
 Wire Wire Line
 	5325 6325 6775 6325
-Wire Wire Line
-	5325 6225 6775 6225
-Wire Wire Line
-	5325 6125 6775 6125
 Connection ~ 3175 6725
 Wire Wire Line
@@
 Wire Wire Line
 	14350 5500 14350 5450
-Wire Bus Line
-	12050 3450 14850 3450
 Wire Wire Line
 	13150 4450 13550 4450
@@
 	12050 3450 12050 6450
 Wire Bus Line
-	13050 3450 13050 4350
+	13050 3450 13050 4550
 Wire Wire Line
 	13150 4350 13550 4350
@@
 Wire Wire Line
 	13150 3650 13550 3650
-Wire Wire Line
-	14350 4350 14750 4350
 Wire Wire Line
 	14350 3750 14750 3750
@@
 Wire Wire Line
 	10650 2750 10650 2800
-Wire Wire Line
-	14900 4150 14900 4450
-Wire Wire Line
-	14900 4450 14350 4450
 Wire Bus Line
-	14850 3450 14850 4250
-Wire Wire Line
-	14350 4150 14900 4150
-Connection ~ 14350 4450
-Connection ~ 14350 4750
-Connection ~ 13550 4850
-Wire Wire Line
-	14350 4850 13550 4850
-Connection ~ 13550 4750
-Connection ~ 13550 4650
-Wire Wire Line
-	13550 4550 13550 4900
-Connection ~ 14350 4650
-Connection ~ 14350 4550
-Wire Wire Line
-	14350 4450 14350 4850
+	14850 3450 14850 3950
 Wire Wire Line
 	5525 7000 5525 6925
@@
 Wire Wire Line
 	6150 7000 6150 6225
-Connection ~ 6150 6225
 Wire Wire Line
 	6250 7000 6250 6125
-Connection ~ 6250 6125
 Wire Wire Line
 	3875 5700 3875 5825
@@
 	7575 8275 7575 8200
 Connection ~ 7875 8200
-Wire Wire Line
-	14350 4250 14750 4250
 $Comp
 L PWR_FLAG #FLG022
@@
 NoConn ~ 9375 4525
 NoConn ~ 9375 4625
+Entry Wire Line
+	13050 4450 13150 4550
+Entry Wire Line
+	13050 4550 13150 4650
+Wire Wire Line
+	13150 4550 13550 4550
+Wire Wire Line
+	13550 4650 13150 4650
+$Comp
+L GND-RESCUE-gpib_adapter #PWR?
+U 1 1 56199A3C
+P 13450 4875
+F 0 "#PWR?" H 13450 4875 30  0001 C CNN
+F 1 "GND" H 13450 4805 30  0001 C CNN
+F 2 "" H 13450 4875 60  0001 C CNN
+F 3 "" H 13450 4875 60  0001 C CNN
+	1    13450 4875
+	1    0    0    -1
+$EndComp
+Wire Wire Line
+	13550 4750 13450 4750
+Wire Wire Line
+	13450 4750 13450 4875
+Wire Wire Line
+	14500 4750 14350 4750
+Wire Wire Line
+	14500 4150 14500 4900
+Wire Wire Line
+	14350 4150 14500 4150
+Connection ~ 14500 4750
+Wire Wire Line
+	14350 4650 14500 4650
+Connection ~ 14500 4650
+Wire Wire Line
+	14350 4550 14500 4550
+Connection ~ 14500 4550
+Wire Wire Line
+	14350 4450 14500 4450
+Connection ~ 14500 4450
+Wire Wire Line
+	14350 4350 14500 4350
+Connection ~ 14500 4350
+Wire Wire Line
+	14350 4250 14500 4250
+Connection ~ 14500 4250
+Wire Bus Line
+	14850 3450 12050 3450
+Wire Wire Line
+	6775 6125 6400 6125
+Wire Wire Line
+	6775 6225 6400 6225
+Wire Wire Line
+	6150 6225 5325 6225
+Wire Wire Line
+	6250 6125 5325 6125
+Text Label 5900 6225 0    60   ~ 0
+TXD
+Text Label 5900 6125 0    60   ~ 0
+RXD
 $EndSCHEMATC

Commit message: fix: fix gpib adapter connections
Parts:
- removed J1: HEADER_2, w_pin_strip:pin_socket_2, symbol HEADER_2
- removed R13, R14, R15, R16, R17, R18, R19, R20: R, Resistors_SMD:R_0805, symbol R-RESCUE-gpib_adapter
- R6: footprint Resistors_SMD:R_2010 -> Resistors_SMD:R_1210
Connections:
- net labels added: _usb+, _usb-, usb+, usb-, usbpwr
- wire segments 219 -> 201
Other:
- moved on the sheet: P2
Changed lines of the file:
@@
 L CONN_5 P2
 U 1 1 4FFF132F
-P 1250 6525
-F 0 "P2" V 1200 6525 50  0000 C CNN
-F 1 "USB" V 1300 6525 50  0000 C CNN
-F 2 "w_conn_pc:conn_usb_B" H 1250 6525 60  0001 C CNN
-F 3 "" H 1250 6525 60  0001 C CNN
-	1    1250 6525
+P 1100 6525
+F 0 "P2" V 1050 6525 50  0000 C CNN
+F 1 "USB" V 1150 6525 50  0000 C CNN
+F 2 "w_conn_pc:conn_usb_B" H 1100 6525 60  0001 C CNN
+F 3 "" H 1100 6525 60  0001 C CNN
+	1    1100 6525
 	-1   0    0    -1
 $EndComp
@@
 Entry Wire Line
 	11950 6550 12050 6450
-Text Label 10075 7300 0    60   ~ 0
-RXD
-Text Label 10075 7200 0    60   ~ 0
-TXD
 $Comp
 L +5V #PWR011
@@
 F 0 "R6" V 2030 6325 50  0000 C CNN
 F 1 "R" V 1950 6325 50  0000 C CNN
-F 2 "Resistors_SMD:R_2010" H 1950 6325 60  0001 C CNN
+F 2 "Resistors_SMD:R_1210" H 1950 6325 60  0001 C CNN
 F 3 "" H 1950 6325 60  0001 C CNN
 	1    1950 6325
@@
 	9675 6425 9775 6525
 Entry Wire Line
-	9775 7100 9875 7200
-Entry Wire Line
-	9775 7200 9875 7300
-Entry Wire Line
 	9675 6525 9775 6625
 Entry Wire Line
@@
 $EndComp
 $Comp
-L R-RESCUE-gpib_adapter R13
-U 1 1 55F59F97
-P 5525 7250
-F 0 "R13" V 5475 7050 50  0000 C CNN
-F 1 "R" V 5525 7250 50  0000 C CNN
-F 2 "Resistors_SMD:R_0805" H 5525 7250 60  0001 C CNN
-F 3 "" H 5525 7250 60  0001 C CNN
-	1    5525 7250
-	1    0    0    -1
-$EndComp
-$Comp
-L R-RESCUE-gpib_adapter R14
-U 1 1 55F59F9D
-P 5625 7250
-F 0 "R14" V 5575 7050 50  0000 C CNN
-F 1 "R" V 5625 7250 50  0000 C CNN
-F 2 "Resistors_SMD:R_0805" H 5625 7250 60  0001 C CNN
-F 3 "" H 5625 7250 60  0001 C CNN
-	1    5625 7250
-	1    0    0    -1
-$EndComp
-$Comp
-L R-RESCUE-gpib_adapter R15
-U 1 1 55F59FA3
-P 5725 7250
-F 0 "R15" V 5675 7050 50  0000 C CNN
-F 1 "R" V 5725 7250 50  0000 C CNN
-F 2 "Resistors_SMD:R_0805" H 5725 7250 60  0001 C CNN
-F 3 "" H 5725 7250 60  0001 C CNN
-	1    5725 7250
-	1    0    0    -1
-$EndComp
-$Comp
-L R-RESCUE-gpib_adapter R16
-U 1 1 55F59FA9
-P 5825 7250
-F 0 "R16" V 5775 7050 50  0000 C CNN
-F 1 "R" V 5825 7250 50  0000 C CNN
-F 2 "Resistors_SMD:R_0805" H 5825 7250 60  0001 C CNN
-F 3 "" H 5825 7250 60  0001 C CNN
-	1    5825 7250
-	1    0    0    -1
-$EndComp
-$Comp
-L R-RESCUE-gpib_adapter R17
-U 1 1 55F59FAF
-P 5950 7250
-F 0 "R17" V 5900 7050 50  0000 C CNN
-F 1 "R" V 5950 7250 50  0000 C CNN
-F 2 "Resistors_SMD:R_0805" H 5950 7250 60  0001 C CNN
-F 3 "" H 5950 7250 60  0001 C CNN
-	1    5950 7250
-	1    0    0    -1
-$EndComp
-$Comp
-L R-RESCUE-gpib_adapter R18
-U 1 1 55F59FB5
-P 6050 7250
-F 0 "R18" V 6000 7050 50  0000 C CNN
-F 1 "R" V 6050 7250 50  0000 C CNN
-F 2 "Resistors_SMD:R_0805" H 6050 7250 60  0001 C CNN
-F 3 "" H 6050 7250 60  0001 C CNN
-	1    6050 7250
-	1    0    0    -1
-$EndComp
-$Comp
-L R-RESCUE-gpib_adapter R19
-U 1 1 55F59FBB
-P 6150 7250
-F 0 "R19" V 6100 7050 50  0000 C CNN
-F 1 "R" V 6150 7250 50  0000 C CNN
-F 2 "Resistors_SMD:R_0805" H 6150 7250 60  0001 C CNN
-F 3 "" H 6150 7250 60  0001 C CNN
-	1    6150 7250
-	1    0    0    -1
-$EndComp
-$Comp
-L R-RESCUE-gpib_adapter R20
-U 1 1 55F59FC1
-P 6250 7250
-F 0 "R20" V 6200 7050 50  0000 C CNN
-F 1 "R" V 6250 7250 50  0000 C CNN
-F 2 "Resistors_SMD:R_0805" H 6250 7250 60  0001 C CNN
-F 3 "" H 6250 7250 60  0001 C CNN
-	1    6250 7250
-	1    0    0    -1
-$EndComp
-$Comp
-L +5V #PWR020
-U 1 1 55F5C6CD
-P 5525 7700
-F 0 "#PWR020" H 5525 7790 20  0001 C CNN
-F 1 "+5V" H 5525 7790 30  0000 C CNN
-F 2 "" H 5525 7700 60  0001 C CNN
-F 3 "" H 5525 7700 60  0001 C CNN
-	1    5525 7700
-	-1   0    0    1
-$EndComp
-$Comp
-L GND-RESCUE-gpib_adapter #PWR021
+L GND-RESCUE-gpib_adapter #PWR020
 U 1 1 55F606F3
 P 7775 7225
-F 0 "#PWR021" H 7775 7225 30  0001 C CNN
+F 0 "#PWR020" H 7775 7225 30  0001 C CNN
 F 1 "GND" H 7775 7155 30  0001 C CNN
 F 2 "" H 7775 7225 60  0001 C CNN
@@
 	1    0    0    -1
 $EndComp
-Connection ~ 5625 7550
-Wire Wire Line
-	5625 7500 5625 7550
-Connection ~ 5725 7550
-Wire Wire Line
-	5725 7550 5725 7500
-Connection ~ 5825 7550
-Wire Wire Line
-	5825 7550 5825 7500
-Connection ~ 5950 7550
-Wire Wire Line
-	5950 7550 5950 7500
-Connection ~ 6050 7550
-Wire Wire Line
-	6050 7550 6050 7500
-Connection ~ 6150 7550
-Wire Wire Line
-	6150 7550 6150 7500
-Connection ~ 5525 7550
-Wire Wire Line
-	6250 7550 6250 7500
-Wire Wire Line
-	5525 7550 6250 7550
-Wire Wire Line
-	5525 7500 5525 7700
 Wire Wire Line
 	6550 6525 6775 6525
@@
 	2200 6325 2350 6325
 Wire Wire Line
-	1700 6325 1650 6325
+	1700 6325 1500 6325
 Wire Wire Line
 	9375 6625 9675 6625
@@
 Wire Wire Line
 	9375 6325 9675 6325
-Wire Wire Line
-	9875 7300 10275 7300
-Wire Wire Line
-	9875 7200 10275 7200
 Wire Wire Line
 	2200 6525 3275 6525
@@
 	14350 6900 14350 6950
 Wire Wire Line
-	1650 6525 1700 6525
+	1500 6525 1700 6525
 Wire Wire Line
 	11550 6550 11950 6550
@@
 Wire Wire Line
 	9200 8750 9200 8650
-Connection ~ 1650 6725
-Wire Wire Line
-	1650 6625 1650 6825
-Wire Wire Line
-	1650 6425 1700 6425
+Connection ~ 1500 6725
+Wire Wire Line
+	1500 6625 1500 6725
+Wire Wire Line
+	1650 6725 1650 6825
+Wire Wire Line
+	1500 6425 1700 6425
 Wire Wire Line
 	9875 6550 10350 6550
@@
 	14850 3450 14850 3950
 Wire Wire Line
-	5525 7000 5525 6925
-Connection ~ 5525 6925
-Wire Wire Line
-	5625 7000 5625 6825
-Connection ~ 5625 6825
-Wire Wire Line
-	5725 7000 5725 6725
-Connection ~ 5725 6725
-Wire Wire Line
-	5825 7000 5825 6625
-Connection ~ 5825 6625
-Wire Wire Line
-	5950 7000 5950 6425
-Connection ~ 5950 6425
-Wire Wire Line
-	6050 7000 6050 6325
-Connection ~ 6050 6325
-Wire Wire Line
-	6150 7000 6150 6225
-Wire Wire Line
-	6250 7000 6250 6125
-Wire Wire Line
 	3875 5700 3875 5825
 Wire Wire Line
@@
 Connection ~ 7875 8200
 $Comp
-L PWR_FLAG #FLG022
+L PWR_FLAG #FLG021
 U 1 1 55F64F5E
 P 2250 6225
-F 0 "#FLG022" H 2250 6320 50  0001 C CNN
+F 0 "#FLG021" H 2250 6320 50  0001 C CNN
 F 1 "PWR_FLAG" H 2250 6405 50  0000 C CNN
 F 2 "" H 2250 6225 60  0000 C CNN
@@
 	6200 4125 6175 4125
 $Comp
-L PWR_FLAG #FLG023
+L PWR_FLAG #FLG022
 U 1 1 55F6B7BB
 P 1775 6725
-F 0 "#FLG023" H 1775 6820 50  0001 C CNN
+F 0 "#FLG022" H 1775 6820 50  0001 C CNN
 F 1 "PWR_FLAG" H 1775 6905 50  0000 C CNN
 F 2 "" H 1775 6725 60  0000 C CNN
@@
 $EndComp
 Wire Wire Line
-	1775 6725 1650 6725
+	1500 6725 1775 6725
 $Comp
 L AVR-ISP-6 CON1
@@
 Wire Wire Line
 	14350 6950 14025 6950
-$Comp
-L HEADER_2 J1
-U 1 1 55F5A829
-P 10375 7250
-F 0 "J1" H 10375 7400 60  0000 C CNN
-F 1 "HEADER_2" H 10375 7100 60  0000 C CNN
-F 2 "w_pin_strip:pin_socket_2" H 10375 7250 60  0001 C CNN
-F 3 "" H 10375 7250 60  0000 C CNN
-	1    10375 7250
-	1    0    0    -1
-$EndComp
 $Comp
 L R-RESCUE-gpib_adapter R25
@@
 	13550 4650 13150 4650
 $Comp
-L GND-RESCUE-gpib_adapter #PWR?
+L GND-RESCUE-gpib_adapter #PWR023
 U 1 1 56199A3C
 P 13450 4875
-F 0 "#PWR?" H 13450 4875 30  0001 C CNN
+F 0 "#PWR023" H 13450 4875 30  0001 C CNN
 F 1 "GND" H 13450 4805 30  0001 C CNN
 F 2 "" H 13450 4875 60  0001 C CNN
@@
 	6775 6225 6400 6225
 Wire Wire Line
-	6150 6225 5325 6225
-Wire Wire Line
-	6250 6125 5325 6125
-Text Label 5900 6225 0    60   ~ 0
+	5800 6225 5325 6225
+Wire Wire Line
+	5800 6125 5325 6125
+Text Label 5800 6225 0    60   ~ 0
 TXD
-Text Label 5900 6125 0    60   ~ 0
+Text Label 5800 6125 0    60   ~ 0
 RXD
+Connection ~ 1650 6725
+Text Label 1550 6325 0    28   ~ 0
+usbpwr
+Text Label 2250 6525 0    60   ~ 0
+usb+
+Text Label 2250 6425 0    60   ~ 0
+usb-
+Text Label 1525 6525 0    28   ~ 0
+_usb+
+Text Label 1525 6425 0    28   ~ 0
+_usb-
 $EndSCHEMATC

Commit message: updating hardware
Parts:
- removed P3: GPIO, w_pin_strip:pin_socket_3x2, symbol CONN_3X2
- removed R10, R11, R12, R9: R, Resistors_SMD:R_0805, symbol R-RESCUE-gpib_adapter
- added C9: 22µ, Capacitors_SMD:c_elec_5x5.3, symbol C-RESCUE-gpib_adapter
- added J1: HEADER_5x2, w_pin_strip:pin_strip_5x2, symbol HEADER_5x2
- C4: footprint Capacitors_SMD:C_1206 -> Capacitors_SMD:C_0805
Connections:
- net +5V: now also C9.1, J1.4
- net ATN: now also U4.41 ((A14)PC6); no longer U4.36 ((A9)PC1)
- net DAV: now also U4.39 ((A12)PC4); no longer U4.38 ((A11)PC3)
- net DIO1: now also U1.12 (D8); no longer U1.19 (D1)
- net DIO1 B: now also U1.9 (B8); no longer U1.2 (B1)
- net DIO2: now also U1.13 (D7); no longer U1.18 (D2)
- net DIO2 B: now also U1.8 (B7); no longer U1.3 (B2)
- net DIO3: now also U1.14 (D6); no longer U1.17 (D3)
- net DIO3 B: now also U1.7 (B6); no longer U1.4 (B3)
- net DIO4: now also U1.15 (D5); no longer U1.16 (D4)
- net DIO4 B: now also U1.6 (B5); no longer U1.5 (B4)
- net DIO5: now also U1.16 (D4); no longer U1.15 (D5)
- net DIO5 B: now also U1.5 (B4); no longer U1.6 (B5)
- net DIO6: now also U1.17 (D3); no longer U1.14 (D6)
- net DIO6 B: now also U1.4 (B3); no longer U1.7 (B6)
- net DIO7: now also U1.18 (D2); no longer U1.13 (D7)
- net DIO7 B: now also U1.3 (B2); no longer U1.8 (B7)
- net DIO8: now also U1.19 (D1); no longer U1.12 (D8)
- net DIO8 B: now also U1.2 (B1); no longer U1.9 (B8)
- net EOI: now also U4.40 ((A13)PC5); no longer U4.37 ((A10)PC2)
- net GND: now also C9.2, J1.10, J1.2
- net IFC: now also U4.36 ((A9)PC1); no longer U4.41 ((A14)PC6)
- net NDAC: now also U4.37 ((A10)PC2); no longer U4.40 ((A13)PC5)
- net NRFD: now also U4.38 ((A11)PC3); no longer U4.39 ((A12)PC4)
- net REN: now also U4.35 ((A8)PC0); no longer U4.42 ((A15/CLK0)PC7)
- net RESET: now also J1.6
- net SRQ: now also U4.42 ((A15/CLK0)PC7); no longer U4.35 ((A8)PC0)
- net TDI: now reaches U4.54 (PF7(ADC7/TDI))
- net TDI: now also J1.9
- net TDO: now reaches U4.55 (PF6(ADC6/TDO))
- net TDO: now also J1.3
- net TMS: now reaches U4.56 (PF5(ADC5/TMS))
- net TMS: now also J1.5
- net TCK: now reaches U4.57 (PF4(ADC4/TCK))
- net TCK: now also J1.1
- net at U4.59 (PF2(ADC2)): no longer R23.1
- net at U4.60 (PF1(ADC1)): no longer R22.1
- net at U4.61 (PF0(ADC0)): no longer R21.1
- net GPIO2: no longer names the net of U4.14 ((OC2A)PB4)
- net GPIO3 renamed PWR
- net PWR: now also R23.1
- net GPIO4 renamed MODE
- net MODE: now also R22.1
- net GPIO5 renamed TALK
- net TALK: now also R21.1
- no-connect marks 16 -> 23
Other:
- moved on the sheet: C1, C3, C4, C5, C6, D1, D2, D3, R21, R22, R23, R25
