File: pcb/gpib_adapter.sch (KiCad schematic (older format))
At the start: 23 parts, among them P1 TC2030-MCP, P2 USB, P5 GPIB, U1 SN75160, U2 SN75161, U3 PIC18(L)F4550-I/PT, X1 8MHz

Commit message: Update pcb files. New version based on pic 18f4550.
Parts:
- added C10: C, Capacitors_SMD:C_1206, symbol C
- added C4, C5: 100n, Capacitors_SMD:C_0805, symbol C
- added C6, C9: 10n, Capacitors_SMD:C_0805, symbol C
- added R7: R, Resistors_SMD:R_1206, symbol R
- P2: footprint w_conn_pc:conn_usb_B -> Connect:USB_B
Connections:
- wire segments 156 -> 170
- no-connect marks 10 -> 11
Changed lines of the file:
@@
 F 0 "P2" V 3075 6050 50  0000 C CNN
 F 1 "USB" V 3175 6050 50  0000 C CNN
-F 2 "w_conn_pc:conn_usb_B" H 3125 6050 60  0001 C CNN
+F 2 "Connect:USB_B" H 3125 6050 60  0001 C CNN
 F 3 "" H 3125 6050 60  0001 C CNN
 	1    3125 6050
@@
 Text Label 5600 4900 2    60   ~ 0
 EOI
-Text Label 8825 6500 2    60   ~ 0
-ATN
-Text Label 8650 4900 2    60   ~ 0
+Text Label 8825 6400 2    60   ~ 0
 SRQ
 $Comp
@@
 Text Label 12500 3400 0    60   ~ 0
 DIO1 B
+Text Label 13650 3400 0    60   ~ 0
+DIO2 B
 Text Label 12500 3500 0    60   ~ 0
-DIO2 B
-Text Label 12500 3600 0    60   ~ 0
 DIO3 B
-Text Label 12500 3700 0    60   ~ 0
+Text Label 13650 3500 0    60   ~ 0
 DIO4 B
-Text Label 13675 3400 0    60   ~ 0
+Text Label 12475 4000 0    60   ~ 0
 DIO5 B
-Text Label 13675 3500 0    60   ~ 0
+Text Label 13625 4000 0    60   ~ 0
 DIO6 B
-Text Label 13675 3600 0    60   ~ 0
+Text Label 12475 4100 0    60   ~ 0
 DIO7 B
-Text Label 13675 3700 0    60   ~ 0
+Text Label 13625 4100 0    60   ~ 0
 DIO8 B
 Entry Wire Line
@@
 Entry Wire Line
 	12300 3900 12400 4000
-Entry Wire Line
-	12300 4000 12400 4100
 Text Label 10850 5600 0    60   ~ 0
 REN B
@@
 Text Label 10850 6300 0    60   ~ 0
 SRQ B
+Text Label 12500 3600 0    60   ~ 0
+EOI B
+Text Label 12500 3700 0    60   ~ 0
+NRFD B
+Text Label 13650 3600 0    60   ~ 0
+DAV B
 Text Label 12500 3800 0    60   ~ 0
-EOI B
-Text Label 12500 4000 0    60   ~ 0
-NRFD B
+IFC B
+Text Label 13650 3800 0    60   ~ 0
+SRQ B
 Text Label 12500 3900 0    60   ~ 0
-DAV B
-Text Label 12500 4200 0    60   ~ 0
-IFC B
-Text Label 12500 4300 0    60   ~ 0
-SRQ B
-Text Label 12500 4400 0    60   ~ 0
 ATN B
-Text Label 12500 4100 0    60   ~ 0
+Text Label 13650 3700 0    60   ~ 0
 NDAC B
 Entry Wire Line
@@
 	1    0    0    -1
 $EndComp
-Text Label 13700 3800 0    60   ~ 0
+Text Label 12475 4200 0    60   ~ 0
 REN B
-Entry Wire Line
-	12300 4100 12400 4200
 Text Label 9350 3300 0    60   ~ 0
 DIO8
@@
 Entry Wire Line
 	9025 4450 9125 4350
-Text Label 8625 5000 2    60   ~ 0
+Text Label 8800 6300 2    60   ~ 0
 ATN
 Entry Wire Line
@@
 	0    1    1    0
 $EndComp
-Entry Wire Line
-	12300 4200 12400 4300
-Entry Wire Line
-	12300 4300 12400 4400
 $Comp
 L GND-RESCUE-gpib_adapter #PWR013
@@
 	8925 5200 9025 5300
 Entry Wire Line
-	8925 6500 9025 6600
-Entry Wire Line
-	8925 4900 9025 5000
-Entry Wire Line
-	8925 5000 9025 5100
+	8925 6300 9025 6400
+Entry Wire Line
+	8925 6400 9025 6500
 $Comp
 L F_Small F1
@@
 Wire Bus Line
 	9025 7825 9025 3150
-Wire Wire Line
-	12400 4200 12800 4200
 Connection ~ 9900 4900
 Connection ~ 9900 2550
@@
 	11300 3200 11300 6200
 Wire Bus Line
-	12300 3200 12300 4300
-Wire Wire Line
-	12400 4100 12800 4100
+	12300 3200 12300 4175
 Wire Wire Line
 	12400 4000 12800 4000
@@
 	9900 2500 9900 2650
 Wire Bus Line
-	14100 3200 14100 3700
+	14100 3200 14100 4100
 Wire Wire Line
 	4375 5850 4375 5550
@@
 	3525 6250 3800 6250
 Wire Wire Line
-	12400 4300 12800 4300
-Wire Wire Line
-	12800 4400 12400 4400
-Wire Wire Line
-	12800 4500 12700 4500
-Wire Wire Line
-	12700 4500 12700 4625
-Wire Wire Line
-	13750 4500 13600 4500
-Wire Wire Line
-	13750 3900 13750 4650
-Wire Wire Line
-	13600 3900 13750 3900
+	12700 4500 12800 4500
+Wire Wire Line
+	12700 4300 12700 4625
+Wire Wire Line
+	13600 4500 13850 4500
 Connection ~ 13750 4500
 Wire Wire Line
-	13600 4400 13750 4400
+	13750 4400 13600 4400
 Connection ~ 13750 4400
 Wire Wire Line
-	13600 4300 13750 4300
+	13600 4300 13850 4300
 Connection ~ 13750 4300
 Wire Wire Line
 	13600 4200 13750 4200
-Connection ~ 13750 4200
-Wire Wire Line
-	13600 4100 13750 4100
-Connection ~ 13750 4100
-Wire Wire Line
-	13600 4000 13750 4000
-Connection ~ 13750 4000
 Wire Bus Line
 	14100 3200 11300 3200
@@
 Wire Wire Line
 	8925 5200 8450 5200
-Wire Wire Line
-	8450 4900 8925 4900
-Wire Wire Line
-	8450 5000 8925 5000
-Wire Wire Line
-	8925 6500 8450 6500
 Wire Wire Line
 	8450 6600 8925 6600
@@
 	0    1    1    0
 $EndComp
-NoConn ~ 8450 6300
-NoConn ~ 8450 6400
+NoConn ~ 8450 4900
+NoConn ~ 8450 5000
 NoConn ~ 6050 6600
 NoConn ~ 6050 6500
@@
 NoConn ~ 6050 5900
 NoConn ~ 6025 8225
+$Comp
+L C C4
+U 1 1 576B0543
+P 2875 8175
+F 0 "C4" H 2925 8275 50  0000 L CNN
+F 1 "100n" H 2925 8075 50  0000 L CNN
+F 2 "Capacitors_SMD:C_0805" H 2875 8175 60  0001 C CNN
+F 3 "" H 2875 8175 60  0001 C CNN
+	1    2875 8175
+	1    0    0    -1
+$EndComp
+$Comp
+L C C5
+U 1 1 576B084B
+P 3250 8175
+F 0 "C5" H 3300 8275 50  0000 L CNN
+F 1 "100n" H 3300 8075 50  0000 L CNN
+F 2 "Capacitors_SMD:C_0805" H 3250 8175 60  0001 C CNN
+F 3 "" H 3250 8175 60  0001 C CNN
+	1    3250 8175
+	1    0    0    -1
+$EndComp
+$Comp
+L C C6
+U 1 1 576B08C8
+P 3575 8175
+F 0 "C6" H 3625 8275 50  0000 L CNN
+F 1 "10n" H 3625 8075 50  0000 L CNN
+F 2 "Capacitors_SMD:C_0805" H 3575 8175 60  0001 C CNN
+F 3 "" H 3575 8175 60  0001 C CNN
+	1    3575 8175
+	1    0    0    -1
+$EndComp
+$Comp
+L C C9
+U 1 1 576B0944
+P 3900 8175
+F 0 "C9" H 3950 8275 50  0000 L CNN
+F 1 "10n" H 3950 8075 50  0000 L CNN
+F 2 "Capacitors_SMD:C_0805" H 3900 8175 60  0001 C CNN
+F 3 "" H 3900 8175 60  0001 C CNN
+	1    3900 8175
+	1    0    0    -1
+$EndComp
+Wire Wire Line
+	2875 8325 2875 8425
+Wire Wire Line
+	2875 8425 3900 8425
+Wire Wire Line
+	3900 8425 3900 8325
+Wire Wire Line
+	3575 8325 3575 8425
+Connection ~ 3575 8425
+Wire Wire Line
+	3250 8325 3250 8550
+Connection ~ 3250 8425
+Wire Wire Line
+	2875 8025 2875 7900
+Wire Wire Line
+	2875 7900 3900 7900
+Wire Wire Line
+	3900 7900 3900 8025
+Wire Wire Line
+	3575 8025 3575 7900
+Connection ~ 3575 7900
+Wire Wire Line
+	3250 7800 3250 8025
+Connection ~ 3250 7900
+$Comp
+L +5V #PWR021
+U 1 1 576B0F5D
+P 3250 7800
+F 0 "#PWR021" H 3250 7890 20  0001 C CNN
+F 1 "+5V" H 3250 7890 30  0000 C CNN
+F 2 "" H 3250 7800 60  0001 C CNN
+F 3 "" H 3250 7800 60  0001 C CNN
+	1    3250 7800
+	1    0    0    -1
+$EndComp
+$Comp
+L GND-RESCUE-gpib_adapter #PWR022
+U 1 1 576B0FEF
+P 3250 8550
+F 0 "#PWR022" H 3250 8550 30  0001 C CNN
+F 1 "GND" H 3250 8480 30  0001 C CNN
+F 2 "" H 3250 8550 60  0001 C CNN
+F 3 "" H 3250 8550 60  0001 C CNN
+	1    3250 8550
+	1    0    0    -1
+$EndComp
+Wire Wire Line
+	13750 4200 13750 4650
+Wire Wire Line
+	12800 4300 12700 4300
+Connection ~ 12700 4500
+Wire Wire Line
+	12800 4400 12700 4400
+Connection ~ 12700 4400
+Entry Wire Line
+	14000 4000 14100 3900
+Entry Wire Line
+	14000 4100 14100 4000
+Wire Wire Line
+	13600 4100 14000 4100
+Wire Wire Line
+	14000 4000 13600 4000
+Entry Wire Line
+	12300 4000 12400 4100
+Entry Wire Line
+	12300 4100 12400 4200
+Wire Wire Line
+	12400 4100 12800 4100
+Wire Wire Line
+	12800 4200 12400 4200
+Wire Wire Line
+	13600 3900 13800 3900
+Wire Wire Line
+	13800 3900 13800 3850
+Wire Wire Line
+	13800 3850 14225 3850
+Wire Wire Line
+	14225 3850 14225 4500
+$Comp
+L C C10
+U 1 1 576C4965
+P 14000 4500
+F 0 "C10" V 14050 4400 50  0000 C CNN
+F 1 "C" V 14050 4575 50  0000 C CNN
+F 2 "Capacitors_SMD:C_1206" H 14038 4350 50  0001 C CNN
+F 3 "" H 14000 4500 50  0000 C CNN
+	1    14000 4500
+	0    1    1    0
+$EndComp
+Wire Wire Line
+	14225 4500 14150 4500
+$Comp
+L R R7
+U 1 1 576C4E2E
+P 14000 4300
+F 0 "R7" V 13950 4150 50  0000 C CNN
+F 1 "R" V 13950 4450 50  0000 C CNN
+F 2 "Resistors_SMD:R_1206" V 13930 4300 50  0001 C CNN
+F 3 "" H 14000 4300 50  0000 C CNN
+	1    14000 4300
+	0    1    1    0
+$EndComp
+Wire Wire Line
+	14150 4300 14225 4300
+Connection ~ 14225 4300
+Wire Wire Line
+	8450 6400 8925 6400
+Wire Wire Line
+	8925 6300 8450 6300
+NoConn ~ 8450 6500
 $EndSCHEMATC

Commit message: change srq to pin rb0 to make it use the external interrupt 0
Changed lines of the file:
@@
 Text Label 5600 4900 2    60   ~ 0
 EOI
-Text Label 8825 6400 2    60   ~ 0
+Text Label 5625 5400 2    60   ~ 0
 SRQ
 $Comp
@@
 Entry Wire Line
 	5350 5400 5250 5500
-Text Label 5575 5400 2    60   ~ 0
+Text Label 8775 6400 2    60   ~ 0
 PE
 Text Label 9325 4350 0    60   ~ 0

Commit message: importing pic18f4550 software
Parts:
- D4: Digikey 568-4140-1-ND -> (none); Vendor Number (none) -> 568-4140-1-ND
- F1: Vendor (none) -> Digikey; Vendor Number (none) -> 507-1485-1-ND
- P2: Vendor (none) -> Digikey; Vendor Number (none) -> 553-2272-ND
- U1: Digikey 296-14950-1-ND -> (none); Vendor (none) -> Digikey; Vendor Number (none) -> 296-14950-1-ND
- U2: Digikey 296-6846-5-ND -> (none); Vendor (none) -> Digikey; Vendor Number (none) -> 296-6846-5-ND
- U3: Digikey PIC18F4550-I/PT-ND -> (none); Vendor (none) -> Digikey; Vendor Id (none) -> PIC18F4550-I/PT-ND
- X1: Digikey 535-9720-1-ND -> (none); Vendor (none) -> Digikey; Vendor Number (none) -> 535-9720-1-ND
Changed lines of the file:
@@
 F 2 "Connect:USB_B" H 3125 6050 60  0001 C CNN
 F 3 "" H 3125 6050 60  0001 C CNN
+F 4 "Digikey" V 3125 6050 60  0001 C CNN "Vendor"
+F 5 "553-2272-ND" V 3125 6050 60  0001 C CNN "Vendor Number"
 	1    3125 6050
 	-1   0    0    -1
@@
 F 2 "Housings_SOIC:SOIC-20_7.5x12.8mm_Pitch1.27mm" H 10200 3750 60  0001 C CNN
 F 3 "datasheets/SN75160B.pdf" H 10200 3750 60  0001 C CNN
-F 4 "296-14950-1-ND" H 10200 3750 60  0001 C CNN "Digikey"
+F 4 "296-14950-1-ND" H 10200 3750 60  0001 C CNN "Vendor Number"
+F 5 "Digikey" H 10200 3750 60  0001 C CNN "Vendor"
 	1    10200 3750
 	1    0    0    -1
@@
 F 2 "Housings_SOIC:SOIC-20_7.5x12.8mm_Pitch1.27mm" H 10200 6050 60  0001 C CNN
 F 3 "datasheets/SN75161B.pdf" H 10200 6050 60  0001 C CNN
-F 4 "296-6846-5-ND" H 10200 6050 60  0001 C CNN "Digikey"
+F 4 "296-6846-5-ND" H 10200 6050 60  0001 C CNN "Vendor Number"
+F 5 "Digikey" H 10200 6050 60  0001 C CNN "Vendor"
 	1    10200 6050
 	1    0    0    -1
@@
 F 2 "Housings_QFP:TQFP-44_10x10mm_Pitch0.8mm" H 7250 6986 50  0001 C CIN
 F 3 "" H 7250 5250 50  0000 C CNN
-F 4 "PIC18F4550-I/PT-ND" H 7250 5500 60  0001 C CNN "Digikey"
+F 4 "PIC18F4550-I/PT-ND" H 7250 5500 60  0001 C CNN "Vendor Id"
+F 5 "Digikey" H 7250 5500 60  0001 C CNN "Vendor"
 	1    7250 5500
 	1    0    0    -1
@@
 F 2 "Resistors_SMD:R_1210" H 3975 5850 50  0001 C CNN
 F 3 "" H 3975 5850 50  0000 C CNN
+F 4 "Digikey" H 3975 5850 60  0001 C CNN "Vendor"
+F 5 "507-1485-1-ND" H 3975 5850 60  0001 C CNN "Vendor Number"
 	1    3975 5850
 	1    0    0    -1
@@
 F 2 "Crystals:Crystal_SMD_5032_4Pads" H 8225 8350 50  0001 C CNN
 F 3 "" H 8225 8350 50  0000 C CNN
-F 4 "535-9720-1-ND" H 8225 8350 60  0001 C CNN "Digikey"
+F 4 "535-9720-1-ND" H 8225 8350 60  0001 C CNN "Vendor Number"
+F 5 "Digikey" H 8225 8350 60  0001 C CNN "Vendor"
 	1    8225 8350
 	1    0    0    -1
@@
 F 2 "esd_protection:PRTR5V0U2X" H 4525 6650 50  0001 C CNN
 F 3 "datasheets/PRTR5V0U2X.pdf" V 4384 6472 50  0001 R CNN
-F 4 "568-4140-1-ND" V 4475 6700 60  0001 C CNN "Digikey"
+F 4 "568-4140-1-ND" V 4475 6700 60  0001 C CNN "Vendor Number"
 	1    4475 6700
 	0    -1   -1   0
